File: Control Board v2/ReflowOvenController/ReflowOvenController.kicad_sch (KiCad schematic)
At the start: 0 parts

Commit message: initial layout
Parts:
- added F1, F2: Fuse, symbol Device:Fuse
- added J1, J2: Conn_Receptacle_3P_Protected, symbol Connector:Conn_Receptacle_3P_Protected
- added J3, J4: Conn_01x01_Socket, symbol Connector:Conn_01x01_Socket
- added SW1: MCU Controlled SSR, symbol Switch:SW_SPST
Connections:
- new net: J2.2 (L), SW1.2 (B)
- new net: F1.1, F2.1, J1.2 (L)
- new net: F2.2, SW1.1 (A)
- new net GNDPWR: J1.3 (PE), J2.3 (PE)
- new net HMI: J4. (Pin_1)
- new net L: F1.2
- new net N: J1.1 (N), J2.1 (N)
- new net Thermocouple: J3. (Pin_1)
Other:
- note added: "120VAC Power"
- note added: "12V AC PSU 36W"
- note added: "12VDC Signal"
- note added: "Digital Bus"
- note added: "Main AC Input"
- note added: "Main Controller PCB"
- note added: "Reflow Oven Controller"
- note added: "Toaster Oven Receptacle"

Commit message: add rev1 files for changing into rev2
Parts:
- F1: value Fuse -> 1A
- F2: value Fuse -> 15A
Other:
- added sheet Controller (controller.kicad_sch)
- added sheet Peripherals (peripherals.kicad_sch)
- added sheet Power Supply (power-supply.kicad_sch)
- added sheet SSR Driver (ssr-driver.kicad_sch)
- note added: "System Overview"
- moved on the sheet: F1, F2
