File: Control Board v2/Reflow-Controller-v2.kicad_sch (KiCad schematic)
At the start: 0 parts

Commit message: Finish preparing the template for v2 design
Other:
- removed sheet Power - Sequencing
- note added: "AC-DC Power Supply"
- note added: "Heater Control"
- note added: "Interface"
- note added: "Microcontroller"
- note removed: "Power - Sequencing"
- note removed: "Random Sheet 1"
- note removed: "Random Sheet 2"
