File: Control Board v2/Reflow-Controller-v2.kicad_pcb (KiCad board)
At the start: 6 copper layers, 0 parts

Commit message: work on PCB layout
Parts:
- added BZ1: CMI-0955-05TH, Buzzer_Beeper:MagneticBuzzer_PUI_AT-0927-TT-6-R, F.Cu at (63.0, 31.5)
- added C1: 100uF, Capacitor_THT:C_Radial_D5.0mm_H5.0mm_P2.00mm, F.Cu at (196.5, 76.5)
- added C2: 10nF 250V, Capacitor_SMD:C_1206_3216Metric_Pad1.33x1.80mm_HandSolder, F.Cu at (187.6, 40.6)
- added C6: 100n, Capacitor_SMD:C_0402_1005Metric, F.Cu at (43.8, 44.9)
- added C7: 100n, Capacitor_SMD:C_0402_1005Metric, F.Cu at (43.8, 46.8)
- added C8: 22p, Capacitor_SMD:C_0402_1005Metric, F.Cu at (43.8, 48.8)
- added C9: 22p, Capacitor_SMD:C_0402_1005Metric, F.Cu at (43.8, 50.8)
- added D1: RED, LED_SMD:LED_0603_1608Metric_Pad1.05x0.95mm_HandSolder, F.Cu at (197.5, 70.0)
- added D2: T2035T-8G-RT, Package_TO_SOT_SMD:TO-263-2, F.Cu at (179.8, 41.9)
- added D3: RED, LED_SMD:LED_0603_1608Metric_Pad1.05x0.95mm_HandSolder, F.Cu at (109.1, 93.1)
- added D4: RED, LED_SMD:LED_0603_1608Metric_Pad1.05x0.95mm_HandSolder, F.Cu at (74.4, 42.3)
- added F1: 1A, Fuse:Fuse_Blade_ATO_directSolder, F.Cu at (153.5, 50.9)
- added F2: 20A, Fuse:Fuse_Blade_ATO_directSolder, F.Cu at (206.3, 24.0)
- added G***: LOGO, LOGO, F.Cu at (162.0, 28.0)
- added H1: MountingHole_Pad, MountingHole:MountingHole_2.7mm_M2.5_Pad_Via, F.Cu at (226.5, 23.5)
- added H2: MountingHole_Pad, MountingHole:MountingHole_2.7mm_M2.5_Pad_Via, F.Cu at (226.5, 122.5)
- added H3: MountingHole_Pad, MountingHole:MountingHole_2.7mm_M2.5_Pad_Via, F.Cu at (133.0, 23.5)
- added H4: MountingHole_Pad, MountingHole:MountingHole_2.7mm_M2.5_Pad_Via, F.Cu at (133.0, 122.5)
- added J1: 1366005, PhoenixContact_SPTA:SPTA-THR 2.53-5.0 P26, F.Cu at (146.2, 40.5)
- added J2: 1366005, PhoenixContact_SPTA:SPTA-THR 2.53-5.0 P26, F.Cu at (213.2, 39.0)
- added J3: ISP, Connector_JST:JST_PH_B6B-PH-K_1x06_P2.00mm_Vertical, F.Cu at (226.5, 97.0)
- added J4: Conn_01x05, Connector_JST:JST_XH_B5B-XH-A_1x05_P2.50mm_Vertical, F.Cu at (134.0, 108.0)
- added J5: Conn_01x14, Connector_PinSocket_2.54mm:PinSocket_1x14_P2.54mm_Vertical, F.Cu at (163.2, 124.0)
- added J6: Conn_01x04, Connector_PinHeader_2.54mm:PinHeader_1x04_P2.54mm_Vertical, F.Cu at (198.5, 83.2)
- added JP1: Jumper_2_Open, Jumper:SolderJumper-2_P1.3mm_Open_RoundedPad1.0x1.5mm, F.Cu at (61.8, 55.7)
- added JP2: Jumper_2_Open, Jumper:SolderJumper-2_P1.3mm_Open_RoundedPad1.0x1.5mm, F.Cu at (61.8, 59.3)
- added PS1: IRM-10-5, Converter_ACDC:Converter_ACDC_MeanWell_IRM-10-xx_THT, F.Cu at (150.3, 80.0)
- added Q1: SQ2315CES-T1_GE3, Package_TO_SOT_SMD:SOT-23_Handsoldering, F.Cu at (62.9, 46.9)
- added Q2: BSS127 H6327, Package_TO_SOT_SMD:SOT-23_Handsoldering, F.Cu at (62.9, 51.7)
- added R1: 330, Resistor_SMD:R_0603_1608Metric_Pad0.98x0.95mm_HandSolder, F.Cu at (197.5, 67.5)
- added R14: 10k, Resistor_SMD:R_0402_1005Metric, F.Cu at (42.2, 60.8)
- added R2: 330, Resistor_SMD:R_2512_6332Metric_Pad1.40x3.35mm_HandSolder, F.Cu at (188.4, 48.1)
- added R3: 330, Resistor_SMD:R_2512_6332Metric_Pad1.40x3.35mm_HandSolder, F.Cu at (193.3, 48.1)
- added R4: 39, Resistor_SMD:R_2512_6332Metric_Pad1.40x3.35mm_HandSolder, F.Cu at (198.2, 48.1)
- added R5: 330, Resistor_SMD:R_0603_1608Metric_Pad0.98x0.95mm_HandSolder, F.Cu at (109.1, 88.0)
- added R6: 330, Resistor_SMD:R_0402_1005Metric, F.Cu at (65.4, 55.0)
- added R7: 330, Resistor_SMD:R_0603_1608Metric_Pad0.98x0.95mm_HandSolder, F.Cu at (109.1, 90.5)
- added R8: 330, Resistor_SMD:R_0603_1608Metric_Pad0.98x0.95mm_HandSolder, F.Cu at (78.7, 42.2)
- added REF**: MTP Logo 5mm Low Detail, Watermarks:MTP Logo 5mm Low Detail, F.Cu at (136.0, 94.5)
- added SW1: SW_SPST, TerminalBlock_Phoenix:TerminalBlock_Phoenix_MKDS-1,5-2-5.08_1x02_P5.08mm_Horizontal, F.Cu at (134.5, 57.0)
- added SW2: SW_Push, Button_Switch_THT:SW_TH_Tactile_Omron_B3F-102x, F.Cu at (222.2, 75.2)
- added TP1: TestPoint, TestPoint:TestPoint_Pad_D1.5mm, F.Cu at (74.0, 35.6)
- added TP2: TestPoint, TestPoint:TestPoint_Pad_D1.5mm, F.Cu at (74.0, 39.2)
- added TP3: TestPoint, TestPoint:TestPoint_Pad_D1.5mm, F.Cu at (77.5, 35.6)
- added TP4: TestPoint, TestPoint:TestPoint_Pad_D1.5mm, F.Cu at (77.5, 39.2)
- added TP5: TestPoint, TestPoint:TestPoint_Pad_D1.5mm, F.Cu at (81.0, 35.6)
- added TP6: TestPoint, TestPoint:TestPoint_Pad_D1.5mm, F.Cu at (81.0, 39.2)
- added TP7: TestPoint, TestPoint:TestPoint_Pad_D1.5mm, F.Cu at (84.6, 35.6)
- added TP8: TestPoint, TestPoint:TestPoint_Pad_D1.5mm, F.Cu at (84.6, 39.2)
- added U2: MOC3083S-TA1, Package_DIP:SMDIP-6_W9.53mm, F.Cu at (207.0, 62.5)
- added U5: ATmega328PB-A, Package_QFP:TQFP-32_7x7mm_P0.8mm, F.Cu at (210.0, 106.5)
- added Y2: 16MHz, Crystal:Crystal_SMD_3225-4Pin_3.2x2.5mm, F.Cu at (43.4, 57.5)
Other:
- board outline added: 102.5 x 108 mm
- board text added: "1"
- board text added: "120VAC AC Power Switch"
- board text added: "14"
- board text added: "1A Blade Fuse"
- board text added: "CS"
- board text added: "GND"
- board text added: "HIGH VOLTAGE"
- board text added: "HIGH VOLTAGE!"
- board text added: "L1"
- board text added: "LCD Connector"
- board text added: "LED"
- board text added: "LOW VOLTAGE"
- board text added: "MISO"
- board text added: "MOSI"
- board text added: "N"
- board text added: "RESET"
- board text added: "RS"
- board text added: "SCK"
- board text added: "T_CS"
- board text added: "T_INT"
- board text added: "T_MISO"
- board text added: "T_MOSI"
- board text added: "T_SCK"
- board text added: "VDD"
- board text removed: "??? ??? ???"
- board text removed: "??? ??? ??? ??? ??? (slot) ??? ??? ??? ??? ???"
- board text removed: "???mm"
- board text removed: "???mm (?oz)"
- board text removed: "???mm ???mm ???mm ???mm ???mm ???mm ???mm ???mm ???mm ???mm"
- board text removed: "ASSEMBLY NOTES (UNLESS OTHERWISE SPECIFIED) 1) DO NOT POPULATE PARTS ARE MARKED WITH A RED CROSS. 2) DO NOT POPULATE PARTS ARE NOT PRESENT IN THE BOM. 3) IF CONFLICTING INFORMATION IS FOUND BETWEEN THE ASSEMBLY FILE AND BOM, BOM SHOULD BE USED AS THE MAIN SOURCE."
- board text removed: "All dimensions are in millimeters unless otherwise specified."
- board text removed: "B.Mask"
- board text removed: "B.Paste"
- board text removed: "B.Silkscreen"
- board text removed: "Back Side"
- board text removed: "Bottom Assembly (Scale 1:1)"
- board text removed: "Bottom Fabrication (Scale 1:1)"
- board text removed: "Bottom Test Points (Scale 1:1)"
- board text removed: "Bottom View"
- board text removed: "Components"
- board text removed: "Copper"
- board text removed: "Core"
- board text removed: "Count"
- board text removed: "Dielectric"
- board text removed: "Dielectric Material"
- board text removed: "Drill Drawing (Top View) (Scale 1:1)"
- board text removed: "F.Mask"
- board text removed: "F.Paste"
- board text removed: "F.Silkscreen"
- board text removed: "FABRICATION NOTES (UNLESS OTHERWISE SPECIFIED) 1) OUTLINE DEFINED IN SEPARATE GERBER FILE WITH {dblquote}Edge_Cuts.GBR{dblquote} SUFFIX. DIMENSIONS OF CIRCUMSIZED RECTANGLE SHOWN ON THIS DWG FOR REF ONLY. 2) SEE SEPARATE DRILL FILES WITH {dblquote}.DRL{dblquote} SUFFIX FOR HOLE LOCATIONS. SELECTED HOLE LOCATIONS SHOWN ON THIS DWG FOR REF ONLY. 3) IMPEDANCE CONTROL REQUIRED. Microstrip 100-Ohm Dif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"
- board text removed: "FR-4"
- board text removed: "Front Side"
- board text removed: "GBR"
- board text removed: "Gerber"
- board text removed: "Hole Size"
- board text removed: "Internal Plane"
- board text removed: "L1 (Sig, PWR)"
- board text removed: "L2 (GND)"
- board text removed: "L3 (Sig, PWR)"
- board text removed: "L4 (Sig, PWR)"
- board text removed: "L5 (GND)"
- board text removed: "L6 (Sig, PWR)"
- board text removed: "Layer"
- board text removed: "Layer Stack Legend"
- board text removed: "Legend"
- board text removed: "Material"
- board text removed: "Net"
- board text removed: "Note: external layer thicknesses are specified after plating."
- board text removed: "PCB3D_BR_BOARDNAME"
- board text removed: "PCB3D_TL_BOARDNAME"
- board text removed: "Paste Mask"
- board text removed: "Plated"
- board text removed: "Plated Plated Plated Plated Plated Plated Plated Plated Plated Unplated"
- board text removed: "Prepreg"
- board text removed: "Ref."
- board text removed: "Signal"
- board text removed: "Solder Mask"
- board text removed: "Solder Resist"
- board text removed: "Symbol"
- board text removed: "THT SMD Total"
- board text removed: "TP? TP? TP?"
- board text removed: "Thickness"
- board text removed: "Top Assembly (Scale 1:1)"
- board text removed: "Top Fabrication (Scale 1:1)"
- board text removed: "Top Test Points (Scale 1:1)"
- board text removed: "Top View"
- board text removed: "Total"
- board text removed: "Total thickness: 1.62mm"
- board text removed: "Type"
- board text removed: "X"
- board text removed: "X [mm]"
- board text removed: "Y"
- board text removed: "Y [mm]"
