File: Control Board v2/Power Board/power-board/Project Architecture.kicad_sch (KiCad schematic)
At the start: 0 parts

Commit message: Import schematics from single-board design
Other:
- sheet Section A - Title A renamed Power Supply
- removed sheet Section B - Title B
- added sheet Heater Control (heater.kicad_sch)
- sheet Power Supply: file Section A - Title A.kicad_sch -> power.kicad_sch
- note added: "Page 3"
- note removed: "Page 5"
