File: Control Board v2/Power Board/power-board/power-board.kicad_sch (KiCad schematic)
At the start: 0 parts

Commit message: Import schematics from single-board design
Other:
- removed sheet Block Diagram
- removed sheet Power - Sequencing
- note added: "Heater Control"
- note added: "Power Supply"
- note removed: "Block Diagram"
- note removed: "Power - Sequencing"
- note removed: "Random Sheet 1"
- note removed: "Random Sheet 2"
