File: Control Board v2/Power Board/power-board/power-board.kicad_pcb (KiCad board)
At the start: 6 copper layers, 0 parts

Commit message: schematic mostly done, start board layout
Parts:
- added C1: 100uF, Capacitor_THT:C_Radial_D5.0mm_H5.0mm_P2.00mm, F.Cu at (174.7, 126.4)
- added C2: 10nF 250V, Capacitor_SMD:C_1206_3216Metric_Pad1.33x1.80mm_HandSolder, F.Cu at (175.7, 63.2)
- added D1: RED, LED_SMD:LED_0603_1608Metric_Pad1.05x0.95mm_HandSolder, F.Cu at (174.6, 131.0)
- added D2: T2035T-8G-RT, Package_TO_SOT_SMD:TO-263-2, F.Cu at (166.2, 64.4)
- added D3: RED, LED_SMD:LED_0603_1608Metric_Pad1.05x0.95mm_HandSolder, F.Cu at (172.0, 114.5)
- added F1: 1A, Fuse:Fuseholder_Clip-5x20mm_Bel_FC-203-22_Lateral_P17.80x5.00mm_D1.17mm_Horizontal, F.Cu at (137.0, 68.1)
- added F2: 20A, Fuse:Fuseholder_Clip-6.3x32mm_Littelfuse_122_Inline_P34.21x7.62mm_D2.54mm_Horizontal, F.Cu at (166.9, 38.0)
- added H1: MountingHole_Pad, MountingHole:MountingHole_2.7mm_M2.5_Pad_Via, F.Cu at (118.0, 27.5)
- added H2: MountingHole_Pad, MountingHole:MountingHole_2.7mm_M2.5_Pad_Via, F.Cu at (201.0, 27.5)
- added H3: MountingHole_Pad, MountingHole:MountingHole_2.7mm_M2.5_Pad_Via, F.Cu at (118.0, 137.0)
- added H4: MountingHole_Pad, MountingHole:MountingHole_2.7mm_M2.5_Pad_Via, F.Cu at (201.0, 137.0)
- added J1: 1366005, PhoenixContact_SPTA:SPTA-THR 2.53-5.0 P26, F.Cu at (131.8, 54.0)
- added J2: 1366005, PhoenixContact_SPTA:SPTA-THR 2.53-5.0 P26, F.Cu at (187.5, 61.0)
- added J6: Conn_01x04, Connector_PinHeader_2.54mm:PinHeader_1x04_P2.54mm_Vertical, F.Cu at (165.5, 125.5)
- added J7: Conn_01x02, TerminalBlock_Phoenix:TerminalBlock_Phoenix_MKDS-1,5-2-5.08_1x02_P5.08mm_Horizontal, F.Cu at (121.0, 122.4)
- added JP3: Jumper_2_Open, Connector_PinHeader_2.54mm:PinHeader_1x02_P2.54mm_Vertical, F.Cu at (170.1, 125.5)
- added PS1: IRM-10-5, Converter_ACDC:Converter_ACDC_MeanWell_IRM-10-xx_THT, F.Cu at (142.5, 96.8)
- added R1: 330, Resistor_SMD:R_0603_1608Metric_Pad0.98x0.95mm_HandSolder, F.Cu at (174.6, 133.6)
- added R2: 330, Resistor_SMD:R_2512_6332Metric_Pad1.40x3.35mm_HandSolder, F.Cu at (162.5, 52.9)
- added R3: 330, Resistor_SMD:R_2512_6332Metric_Pad1.40x3.35mm_HandSolder, F.Cu at (167.4, 52.9)
- added R4: 39, Resistor_SMD:R_2512_6332Metric_Pad1.40x3.35mm_HandSolder, F.Cu at (172.3, 52.9)
- added R5: 330, Resistor_SMD:R_0603_1608Metric_Pad0.98x0.95mm_HandSolder, F.Cu at (167.6, 114.4)
- added R7: 330, Resistor_SMD:R_0603_1608Metric_Pad0.98x0.95mm_HandSolder, F.Cu at (167.6, 116.9)
- added RV1: TMOV20RP150E, Varistor:RV_Disc_D21.5mm_W8.4mm_P10mm, F.Cu at (139.0, 58.0)
- added SW1: SW_SPST, TerminalBlock_Phoenix:TerminalBlock_Phoenix_MKDS-1,5-2-5.08_1x02_P5.08mm_Horizontal, F.Cu at (120.8, 83.0)
- added U2: MOC3083S-TA1, Package_DIP:SMDIP-6_W9.53mm, F.Cu at (187.2, 115.5)
Other:
- board outline added: 92 x 118.5 mm
- board text removed: "??? ??? ???"
- board text removed: "??? ??? ??? ??? ??? (slot) ??? ??? ??? ??? ???"
- board text removed: "???mm"
- board text removed: "???mm (?oz)"
- board text removed: "???mm ???mm ???mm ???mm ???mm ???mm ???mm ???mm ???mm ???mm"
- board text removed: "ASSEMBLY NOTES (UNLESS OTHERWISE SPECIFIED) 1) DO NOT POPULATE PARTS ARE MARKED WITH A RED CROSS. 2) DO NOT POPULATE PARTS ARE NOT PRESENT IN THE BOM. 3) IF CONFLICTING INFORMATION IS FOUND BETWEEN THE ASSEMBLY FILE AND BOM, BOM SHOULD BE USED AS THE MAIN SOURCE."
- board text removed: "All dimensions are in millimeters unless otherwise specified."
- board text removed: "B.Mask"
- board text removed: "B.Paste"
- board text removed: "B.Silkscreen"
- board text removed: "Back Side"
- board text removed: "Bottom Assembly (Scale 1:1)"
- board text removed: "Bottom Fabrication (Scale 1:1)"
- board text removed: "Bottom Test Points (Scale 1:1)"
- board text removed: "Bottom View"
- board text removed: "Components"
- board text removed: "Copper"
- board text removed: "Core"
- board text removed: "Count"
- board text removed: "Dielectric"
- board text removed: "Dielectric Material"
- board text removed: "Drill Drawing (Top View) (Scale 1:1)"
- board text removed: "F.Mask"
- board text removed: "F.Paste"
- board text removed: "F.Silkscreen"
- board text removed: "FABRICATION NOTES (UNLESS OTHERWISE SPECIFIED) 1) OUTLINE DEFINED IN SEPARATE GERBER FILE WITH {dblquote}Edge_Cuts.GBR{dblquote} SUFFIX. DIMENSIONS OF CIRCUMSIZED RECTANGLE SHOWN ON THIS DWG FOR REF ONLY. 2) SEE SEPARATE DRILL FILES WITH {dblquote}.DRL{dblquote} SUFFIX FOR HOLE LOCATIONS. SELECTED HOLE LOCATIONS SHOWN ON THIS DWG FOR REF ONLY. 3) IMPEDANCE CONTROL REQUIRED. Microstrip 100-Ohm Dif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"
- board text removed: "FR-4"
- board text removed: "Front Side"
- board text removed: "GBR"
- board text removed: "Gerber"
- board text removed: "Hole Size"
- board text removed: "Internal Plane"
- board text removed: "L1 (Sig, PWR)"
- board text removed: "L2 (GND)"
- board text removed: "L3 (Sig, PWR)"
- board text removed: "L4 (Sig, PWR)"
- board text removed: "L5 (GND)"
- board text removed: "L6 (Sig, PWR)"
- board text removed: "Layer"
- board text removed: "Layer Stack Legend"
- board text removed: "Legend"
- board text removed: "Material"
- board text removed: "Net"
- board text removed: "Note: external layer thicknesses are specified after plating."
- board text removed: "PCB3D_BR_BOARDNAME"
- board text removed: "PCB3D_TL_BOARDNAME"
- board text removed: "Paste Mask"
- board text removed: "Plated"
- board text removed: "Plated Plated Plated Plated Plated Plated Plated Plated Plated Unplated"
- board text removed: "Prepreg"
- board text removed: "Ref."
- board text removed: "Signal"
- board text removed: "Solder Mask"
- board text removed: "Solder Resist"
- board text removed: "Symbol"
- board text removed: "THT SMD Total"
- board text removed: "TP? TP? TP?"
- board text removed: "Thickness"
- board text removed: "Top Assembly (Scale 1:1)"
- board text removed: "Top Fabrication (Scale 1:1)"
- board text removed: "Top Test Points (Scale 1:1)"
- board text removed: "Top View"
- board text removed: "Total"
- board text removed: "Total thickness: 1.62mm"
- board text removed: "Type"
- board text removed: "X"
- board text removed: "X [mm]"
- board text removed: "Y"
- board text removed: "Y [mm]"
