File: Revision 3/Hardware/Power Board/powerBoard/heater.kicad_sch (KiCad schematic)
At the start: 12 parts, among them J2 1366005, J3 Conn_01x03, U2 MOC3083S-TA1

Commit message: Revise project structure
Parts:
- J3: footprint Connector_PinHeader_2.54mm:PinHeader_1x03_P2.54mm_Vertical -> Connector_JST:JST_PH_B3B-PH-K_1x03_P2.00mm_Vertical
Changed lines of the file:
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@@
 			)
 		)
-		(property "Footprint" "Connector_PinHeader_2.54mm:PinHeader_1x03_P2.54mm_Vertical"
+		(property "Footprint" "Connector_JST:JST_PH_B3B-PH-K_1x03_P2.00mm_Vertical"
 			(at 92.71 156.21 0)
 			(effects
