File: Revision 3/Hardware/TC Front End/front-end/front-end.kicad_pcb (KiCad board)
At the start: 6 copper layers, 0 parts

Commit message: Project template fully initialized
Other:
- board text removed: "??? ??? ???"
- board text removed: "??? ??? ??? ??? ??? (slot) ??? ??? ??? ??? ???"
- board text removed: "???mm"
- board text removed: "???mm (?oz)"
- board text removed: "???mm ???mm ???mm ???mm ???mm ???mm ???mm ???mm ???mm ???mm"
- board text removed: "ASSEMBLY NOTES (UNLESS OTHERWISE SPECIFIED) 1) DO NOT POPULATE PARTS ARE MARKED WITH A RED CROSS. 2) DO NOT POPULATE PARTS ARE NOT PRESENT IN THE BOM. 3) IF CONFLICTING INFORMATION IS FOUND BETWEEN THE ASSEMBLY FILE AND BOM, BOM SHOULD BE USED AS THE MAIN SOURCE."
- board text removed: "All dimensions are in millimeters unless otherwise specified."
- board text removed: "B.Mask"
- board text removed: "B.Paste"
- board text removed: "B.Silkscreen"
- board text removed: "Back Side"
- board text removed: "Bottom Assembly (Scale 1:1)"
- board text removed: "Bottom Fabrication (Scale 1:1)"
- board text removed: "Bottom Test Points (Scale 1:1)"
- board text removed: "Bottom View"
- board text removed: "Components"
- board text removed: "Copper"
- board text removed: "Core"
- board text removed: "Count"
- board text removed: "Dielectric"
- board text removed: "Dielectric Material"
- board text removed: "Drill Drawing (Top View) (Scale 1:1)"
- board text removed: "F.Mask"
- board text removed: "F.Paste"
- board text removed: "F.Silkscreen"
- board text removed: "FABRICATION NOTES (UNLESS OTHERWISE SPECIFIED) 1) OUTLINE DEFINED IN SEPARATE GERBER FILE WITH {dblquote}Edge_Cuts.GBR{dblquote} SUFFIX. DIMENSIONS OF CIRCUMSIZED RECTANGLE SHOWN ON THIS DWG FOR REF ONLY. 2) SEE SEPARATE DRILL FILES WITH {dblquote}.DRL{dblquote} SUFFIX FOR HOLE LOCATIONS. SELECTED HOLE LOCATIONS SHOWN ON THIS DWG FOR REF ONLY. 3) IMPEDANCE CONTROL REQUIRED. Microstrip 100-Ohm Dif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"
- board text removed: "FR-4"
- board text removed: "Front Side"
- board text removed: "GBR"
- board text removed: "Gerber"
- board text removed: "Hole Size"
- board text removed: "Internal Plane"
- board text removed: "L1 (Sig, PWR)"
- board text removed: "L2 (GND)"
- board text removed: "L3 (Sig, PWR)"
- board text removed: "L4 (Sig, PWR)"
- board text removed: "L5 (GND)"
- board text removed: "L6 (Sig, PWR)"
- board text removed: "Layer"
- board text removed: "Layer Stack Legend"
- board text removed: "Legend"
- board text removed: "Material"
- board text removed: "Net"
- board text removed: "Note: external layer thicknesses are specified after plating."
- board text removed: "PCB3D_BR_BOARDNAME"
- board text removed: "PCB3D_TL_BOARDNAME"
- board text removed: "Paste Mask"
- board text removed: "Plated"
- board text removed: "Plated Plated Plated Plated Plated Plated Plated Plated Plated Unplated"
- board text removed: "Prepreg"
- board text removed: "Ref."
- board text removed: "Signal"
- board text removed: "Solder Mask"
- board text removed: "Solder Resist"
- board text removed: "Symbol"
- board text removed: "THT SMD Total"
- board text removed: "TP? TP? TP?"
- board text removed: "Thickness"
- board text removed: "Top Assembly (Scale 1:1)"
- board text removed: "Top Fabrication (Scale 1:1)"
- board text removed: "Top Test Points (Scale 1:1)"
- board text removed: "Top View"
- board text removed: "Total"
- board text removed: "Total thickness: 1.62mm"
- board text removed: "Type"
- board text removed: "X"
- board text removed: "X [mm]"
- board text removed: "Y"
- board text removed: "Y [mm]"
