File: Revision 3/Hardware/TC Front End/front-end/front-end.kicad_pcb (KiCad board)
At the start: 6 copper layers, 0 parts

Commit message: Add parts to PCB and get models. Layout can now begin
Parts:
- added C1: 104, Capacitor_SMD:C_0603_1608Metric_Pad1.08x0.95mm_HandSolder, F.Cu at (155.7, 106.8)
- added D1: BZT52C4V7-13-F, Diode_SMD:D_SOD-123, F.Cu at (165.9, 107.2)
- added D2: BZT52C4V7-13-F, Diode_SMD:D_SOD-123, F.Cu at (165.9, 110.6)
- added J1: Conn_01x02, TerminalBlock_Phoenix:TerminalBlock_Phoenix_MKDS-1,5-2_1x02_P5.00mm_Horizontal, F.Cu at (131.5, 119.7)
- added J2: 4DB-P108-02, 4DB_P108_02:CONN_4DB-P108-02_TEC, F.Cu at (130.5, 102.0)
- added J5: Conn_01x04, Connector_PinHeader_2.54mm:PinHeader_1x04_P2.54mm_Vertical, F.Cu at (179.5, 100.9)
- added R1: 1k, Resistor_SMD:R_0603_1608Metric_Pad0.98x0.95mm_HandSolder, F.Cu at (155.7, 109.3)
- added R2: TC33X-2-103E, Potentiometer_SMD:Potentiometer_Bourns_TC33X_Vertical, F.Cu at (150.5, 100.8)
- added R3: 15k, Resistor_SMD:R_0603_1608Metric_Pad0.98x0.95mm_HandSolder, F.Cu at (155.7, 111.8)
- added R4: 560, Resistor_SMD:R_0603_1608Metric_Pad0.98x0.95mm_HandSolder, F.Cu at (155.7, 114.3)
- added R5: TC33X-2-102E, Potentiometer_SMD:Potentiometer_Bourns_TC33X_Vertical, F.Cu at (150.5, 105.5)
- added R6: TC33X-2-103E, Potentiometer_SMD:Potentiometer_Bourns_TC33X_Vertical, F.Cu at (150.5, 110.3)
- added R7: 15k, Resistor_SMD:R_0603_1608Metric_Pad0.98x0.95mm_HandSolder, F.Cu at (155.7, 116.8)
- added R8: 560, Resistor_SMD:R_0603_1608Metric_Pad0.98x0.95mm_HandSolder, F.Cu at (155.7, 119.3)
- added R9: TC33X-2-102E, Potentiometer_SMD:Potentiometer_Bourns_TC33X_Vertical, F.Cu at (150.5, 115.0)
- added U1: LM321, Package_TO_SOT_SMD:SOT-23-5, F.Cu at (160.4, 107.9)
- added U2: LM321, Package_TO_SOT_SMD:SOT-23-5, F.Cu at (160.4, 112.6)
- added U3: DS18B20+, Package_TO_SOT_THT:TO-92_Inline, F.Cu at (165.0, 115.5)
Other:
- board outline added: 65 x 35 mm
